Commit message: use `stl`

File: unnamed/submodels/serial_abstract/urdf/serial_abstract.urdf (robot description, URDF)
Before this commit: robot serial_abstract, 3 links, 2 joints
Links:
- link Robotic_Collaborative_Robot_Arm_EB-052_link: geometry visual mesh filename=package://serial_abstract/../../meshes/stl/Robotic_Collabor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 scale=1.00000 1.00000 1.00000
- link Robotic_Collaborative_Robot_Arm_EB-108_link: geometry visual mesh filename=package://serial_abstract/../../meshes/stl/Robotic_Collabor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 scale=1.00000 1.00000 1.00000
- link new_link: geometry visual mesh filename=package://serial_abstract/../../meshes/stl/Robotic_Collabor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 scale=1.00000 1.00000 1.00000; visual mesh filename=package://serial_abstract/../../meshes/stl/Robotic_Collabor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 scale=1.00000 1.00000 1.00000

File: unnamed/urdf/unnamed.urdf (robot description, URDF)
Before this commit: robot unnamed, 3 links, 2 joints
Links:
- link Robotic_Collaborative_Robot_Arm_EB-052_link: geometry visual mesh filename=package://my_package/meshes/stl/Robotic_Collaborative_Robot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 scale=1.00000 1.00000 1.00000
- link Robotic_Collaborative_Robot_Arm_EB-108_link: geometry visual mesh filename=package://my_package/meshes/stl/Robotic_Collaborative_Robot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 scale=1.00000 1.00000 1.00000
- link new_link: geometry visual mesh filename=package://my_package/meshes/stl/Robotic_Collaborative_Robot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 scale=1.00000 1.00000 1.00000; visual mesh filename=package://my_package/meshes/stl/Robotic_Collaborative_Robot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 scale=1.00000 1.00000 1.00000
